File: Project/dualScaleBoard_HX711.sch (EAGLE design)
At the start: 43 parts, among them Q1 MMBT4403, Q2 MMBT4403, U1 HX711, U2 HX711

Commit message: BOM update
Parts:
- C1, C12, C2, C3, C4, C6, C8, C9: LCSC (none) -> C1591
- C10, C11, C13, C14, C5, C7: LCSC (none) -> C19702
- L1, L2: LCSC (none) -> C275346
- Q1, Q2: LCSC (none) -> C78864
- R1, R2, R3, R4: LCSC (none) -> C328416
- R10, R9: LCSC (none) -> C317926
- R5: LCSC (none) -> C351700
- R6, R8: LCSC (none) -> C517526
- R7: value 20K -> 20k; LCSC (none) -> C351700
- U1, U2: LCSC (none) -> C43656

Commit message: VDD LDO option
Parts:
- added IC1: MCP1700T, linear:MCP1703CB
Connections:
- net GND: now also IC1.GND
- net VCC: now also IC1.VI
- net VDD: now also IC1.VO
Changed lines of the file:
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@@
 <part name="U$1" library="adafruit" library_urn="urn:adsk.eagle:library:420" deviceset="FIDUCIAL" device="" package3d_urn="urn:adsk.eagle:package:6240632/1"/>
 <part name="U$2" library="adafruit" library_urn="urn:adsk.eagle:library:420" deviceset="FIDUCIAL" device="" package3d_urn="urn:adsk.eagle:package:6240632/1"/>
+<part name="IC1" library="linear" library_urn="urn:adsk.eagle:library:262" deviceset="MCP1703" device="CB" package3d_urn="urn:adsk.eagle:package:16489/2" value="MCP1700T">
+<attribute name="LCSC" value="C39051"/>
+</part>
+<part name="SUPPLY9" library="Power_Symbols" library_urn="urn:adsk.eagle:library:16502351" deviceset="GND-BAR" device="" value="GND"/>
 </parts>
 <sheets>
@@
 <instance part="U$1" gate="G$1" x="243.84" y="40.64" smashed="yes"/>
 <instance part="U$2" gate="G$1" x="238.76" y="40.64" smashed="yes"/>
+<instance part="IC1" gate="G$1" x="208.28" y="93.98" smashed="yes">
+<attribute name="NAME" x="200.66" y="99.695" size="1.778" layer="95"/>
+<attribute name="VALUE" x="200.66" y="97.155" size="1.778" layer="96"/>
+<attribute name="LCSC" x="208.28" y="93.98" size="1.778" layer="96" display="off"/>
+</instance>
+<instance part="SUPPLY9" gate="G$1" x="208.28" y="78.74" smashed="yes">
+<attribute name="VALUE" x="208.28" y="76.835" size="1.778" layer="96" align="center"/>
+</instance>
 </instances>
 <busses>
@@
 <label x="193.04" y="53.34" size="1.778" layer="95"/>
 </segment>
+<segment>
+<pinref part="IC1" gate="G$1" pin="VO"/>
+<wire x1="218.44" y1="93.98" x2="228.6" y2="93.98" width="0.1524" layer="91"/>
+<label x="223.52" y="93.98" size="1.778" layer="95"/>
+</segment>
 </net>
 <net name="N$1" class="0">
@@
 <wire x1="213.36" y1="58.42" x2="226.06" y2="58.42" width="0.1524" layer="91"/>
 <label x="220.98" y="58.42" size="1.778" layer="95"/>
+</segment>
+<segment>
+<pinref part="IC1" gate="G$1" pin="VI"/>
+<wire x1="198.12" y1="93.98" x2="187.96" y2="93.98" width="0.1524" layer="91"/>
+<label x="187.96" y="93.98" size="1.778" layer="95"/>
 </segment>
 </net>
@@
 <label x="220.98" y="55.88" size="1.778" layer="95"/>
 </segment>
-</net>
+<segment>
+<pinref part="SUPPLY9" gate="G$1" pin="GND"/>
+<pinref part="IC1" gate="G$1" pin="GND"/>
+<wire x1="208.28" y1="81.28" x2="208.28" y2="86.36" width="0.1524" layer="91"/>
+</segment>
+</net>

Commit message: pin reassignment
Connections:
- net DOUT1: now also JP1.2
- net DOUT2: now also JP1.10
- net VCC: now also JP1.7; no longer JP1.4
- net VDD: now also JP1.4; no longer JP1.7
Changed lines of the file:
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@@
-</segment>
-<segment>
-<pinref part="JP1" gate="A" pin="7"/>
-<wire x1="205.74" y1="53.34" x2="193.04" y2="53.34" width="0.1524" layer="91"/>
-<label x="193.04" y="53.34" size="1.778" layer="95"/>
 </segment>
 <segment>
@@
 <wire x1="218.44" y1="93.98" x2="228.6" y2="93.98" width="0.1524" layer="91"/>
 <label x="223.52" y="93.98" size="1.778" layer="95"/>
+</segment>
+<segment>
+<pinref part="JP1" gate="A" pin="4"/>
+<wire x1="213.36" y1="58.42" x2="226.06" y2="58.42" width="0.1524" layer="91"/>
+<label x="220.98" y="58.42" size="1.778" layer="95"/>
 </segment>
 </net>
@@
 </segment>
 <segment>
-<pinref part="JP1" gate="A" pin="4"/>
-<wire x1="213.36" y1="58.42" x2="226.06" y2="58.42" width="0.1524" layer="91"/>
-<label x="220.98" y="58.42" size="1.778" layer="95"/>
-</segment>
-<segment>
 <pinref part="IC1" gate="G$1" pin="VI"/>
 <wire x1="198.12" y1="93.98" x2="187.96" y2="93.98" width="0.1524" layer="91"/>
 <label x="187.96" y="93.98" size="1.778" layer="95"/>
+</segment>
+<segment>
+<pinref part="JP1" gate="A" pin="7"/>
+<wire x1="205.74" y1="53.34" x2="193.04" y2="53.34" width="0.1524" layer="91"/>
+<label x="193.04" y="53.34" size="1.778" layer="95"/>
 </segment>
 </net>
@@
 <label x="193.04" y="60.96" size="1.778" layer="95"/>
 </segment>
+<segment>
+<pinref part="JP1" gate="A" pin="2"/>
+<wire x1="213.36" y1="60.96" x2="226.06" y2="60.96" width="0.1524" layer="91"/>
+<label x="218.44" y="60.96" size="1.778" layer="95"/>
+</segment>
 </net>
 <net name="N$21" class="0">
@@
 <label x="114.3" y="50.8" size="1.778" layer="95"/>
 </segment>
-</net>
+<segment>
+<pinref part="JP1" gate="A" pin="10"/>
+<wire x1="213.36" y1="50.8" x2="226.06" y2="50.8" width="0.1524" layer="91"/>
+<label x="218.44" y="50.8" size="1.778" layer="95"/>
+</segment>
+</net>

Commit message: FPC version
Parts:
- removed JP1: (no value), pinhead:PINHD-2X5
- removed JP10, JP11: JUMPER-SMT_2_NC_TRACE_SILK, SparkFun-Jumpers:JUMPER-SMT_2_NC_TRACE_SILK
- added J1: 687110149022, Wurth_Connectors_WR-FPC:6871XX149022_687110149022
Connections:
- net DOUT1: now also J1.2; no longer JP1.1, JP1.2
- net DOUT2: now also J1.9; no longer JP1.10, JP1.9
- net GND: now also J1.1, J1.10, J1.5, J1.6, J1.Z1, J1.Z2; no longer JP1.5, JP1.6
- net SCK1: now also J1.4; no longer JP1.3, JP10.2
- net SCK2: now also J1.7; no longer JP1.8, JP10.1
- net VCC: now also J1.3, J1.8; no longer JP1.7, JP11.1
- net VDD: no longer JP1.4, JP11.2
